File: 0027_Rain_Detection_Module_LM393.kicad_sch (KiCad schematic)
At the start: 10 parts, among them J1 Screw_Terminal_01x02, U2 LM393D

Commit message: Add files via upload
Parts:
- added J2: Screw_Terminal_01x02, Library:rain, symbol Connector:Screw_Terminal_01x02
- added U1: ~, Moduler_:pin_header, symbol moduler_pin:air
- C1, C2: footprint (none) -> Capacitor_SMD:C_0805_2012Metric
- D1, D2: footprint (none) -> LED_SMD:LED_0805_2012Metric
- J1: footprint (none) -> TerminalBlock_4Ucon:TerminalBlock_4Ucon_1x02_P3.50mm_Horizontal
- R1, R2, R3: footprint (none) -> Resistor_SMD:R_0805_2012Metric
- RV1: footprint (none) -> meminle:3362P_1
- U2: footprint SOIC127P599X175-8N -> LM393:SOIC127P599X175-8N
Connections:
- net DOUT: now also U1.12
- net GND: now also RV1.1, J2.2 (Pin_2), U1.9; no longer RV1.3
- net AOUT: now reaches J1.1 (Pin_1), R2.2
- net AOUT: now also C2.1, U2.5 (2IN+), J2.1 (Pin_1), U1.13
- net VCC renamed +3V3
- net +3V3: now also RV1.3, U1.8; no longer C2.1, RV1.1, U2.5 (2IN+)
- no-connect marks 3 -> 17
Other:
- note added: "AIR PIN"
- note added: "SENSOR"
- moved on the sheet: C1, C2, D1, D2, J1, R1, R2, R3, U2
